File: SquareSprite.sch (EAGLE design)
At the start: 24 parts, among them P1 SPRITE_PIN, P2 SPRITE_PIN, U1 CC430F5137, X1 TCXO_7Z

Commit message: New sprite with spring
Parts:
- removed U$1: FASTCAP, FastCap:FASTCAP
- added C10: 10uF, SparkFun:CAP0603-CAP
- added C7: 10nF, SparkFun:CAP0603-CAP
- added C8, C9: 0.1uF, SparkFun:CAP0603-CAP
- added U2: LSM9DS1, LSM9DS1:LSM9DS1
Connections:
- new net N$5: C7.1, U2.CAP
- new net N$6: C8.1, U2.C1
- net GND: now also C10.2, C7.2, C8.2, C9.2, P1.PIN, U2.GND, U2.RES; no longer P2.PIN, U$1.-
- net SCL: now also U2.SCL/SPC
- net SDA: now also U2.SDA/SDI/SDO
- net VCC: now also C10.1, C9.1, P2.PIN, U2.CS_A/G, U2.CS_M, U2.SDO_A/G, U2.SDO_M, U2.VDD, U2.VDDIO; no longer P1.PIN, U$1.+
Other:
- moved on the sheet: C1, C2, C3, C4, C5, C6, D1, JP2, JP3, L1, R1, R2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
